File: kicad/i2c-adapter.kicad_sch (KiCad schematic)
At the start: 46 parts, among them J1 Conn_02x13_Top_Bottom, J10 AUX IN, J11 +5V, J2 I2C-1, J3 I2C-2, J4 I2C-3, J5 I2C-4, J6 SPI-1, J7 SPI-2, J8 SPI-3, J9 SPI-4, U1 74HC05, U2 74HC244, U3 LM1117-3.3

Commit message: With the help of @K3130440, I've added level shifters to the 3V3 data lines and a 74HC138 which adds more Chip Select lines (that are then routed to the EyeSPI connector). Updated Schematic PDF to include the hardware changes. I moved the major ICs closer together to save on board space. Current Board size: 98 x 66.3; Via count: 52; I tried to make sure many components have a position as close to a whole number as possible. Added 3D models to shorten the height of the I2C/SPI proto area. Updated the chips to have a stacked 3D Models structure and added text to each chip. Updated 3D render with the updated 3D Models. Quite a few of the .asm files in src/ need to be updated with the hardware changes.
Parts:
- removed R12: 330, Resistor_SMD:R_0805_2012Metric_Pad1.20x1.40mm_HandSolder, symbol Device:R
- added C17: 0.1uF, Capacitor_SMD:C_0805_2012Metric_Pad1.18x1.45mm_HandSolder, symbol Device:C_Small
- added Q1, Q2, Q3, Q4, Q5: BSS138, Package_TO_SOT_SMD:SOT-23, symbol Transistor_FET:BSS138
- added R13, R14, R15, R16, R17, R18, R19, R20: 10K, Resistor_SMD:R_0805_2012Metric_Pad1.20x1.40mm_HandSolder, symbol Device:R_Small
- added R21, R22, R23, R24, R25, R26: 2K7, Resistor_SMD:R_0805_2012Metric_Pad1.20x1.40mm_HandSolder, symbol Device:R
- added R27, R28, R29, R30, R31, R32: 4K7, Resistor_SMD:R_0805_2012Metric_Pad1.20x1.40mm_HandSolder, symbol Device:R
- added U4: 74HC138, Package_DIP:DIP-16_W7.62mm_Socket, symbol EasyEDA:SN74HC138N
- C1: Digi-Key_PN (none) -> 1276-2872-1-ND; LCSC C15850 -> C95841; MPN (none) -> CL21B106KOQNNNE; Manufacturer (none) -> Samsung Electro-Mechanics
- C10: renamed from C9; Digi-Key_PN (none) -> 1276-1180-1-ND; LCSC C28233 -> C136621; MPN (none) -> CL21B104KBFNNNE; Manufacturer (none) -> Samsung Electro-Mechanics
- C11: renamed from C10; Digi-Key_PN (none) -> 1276-1180-1-ND; LCSC C28233 -> C136621; MPN (none) -> CL21B104KBFNNNE; Manufacturer (none) -> Samsung Electro-Mechanics
- C12: renamed from C11; Digi-Key_PN (none) -> 1276-1180-1-ND; LCSC C28233 -> C136621; MPN (none) -> CL21B104KBFNNNE; Manufacturer (none) -> Samsung Electro-Mechanics
- C13: renamed from C12; Digi-Key_PN (none) -> 1276-1180-1-ND; LCSC C28233 -> C136621; MPN (none) -> CL21B104KBFNNNE; Manufacturer (none) -> Samsung Electro-Mechanics
- C14: renamed from C15; Digi-Key_PN 1276-1935-1-ND -> 1276-1180-1-ND; LCSC C28233 -> C136621; MPN CL10B104KB8NNWC -> CL21B104KBFNNNE
- C15: renamed from C13; Digi-Key_PN (none) -> 1276-1180-1-ND; LCSC C28233 -> C136621; MPN (none) -> CL21B104KBFNNNE; Manufacturer (none) -> Samsung Electro-Mechanics
- C16: renamed from C4; Digi-Key_PN (none) -> 1276-1180-1-ND; LCSC C28233 -> C136621; MPN (none) -> CL21B104KBFNNNE; Manufacturer (none) -> Samsung Electro-Mechanics
- C2: renamed from C14; Digi-Key_PN P975-ND -> 1276-2872-1-ND; LCSC C15850 -> C95841; MPN ECE-A1EKS100 -> CL21B106KOQNNNE; Manufacturer Panasonic Electronic Components -> Samsung Electro-Mechanics
- C3: renamed from C16; Digi-Key_PN 1276-1298-1-ND -> 1276-2872-1-ND; LCSC C15850 -> C95841; MPN CL21A106MQFNNNE -> CL21B106KOQNNNE
- C4: renamed from C2; Digi-Key_PN (none) -> 1276-1180-1-ND; LCSC C28233 -> C136621; MPN (none) -> CL21B104KBFNNNE; Manufacturer (none) -> Samsung Electro-Mechanics
- C5: renamed from C3; Digi-Key_PN (none) -> 1276-1180-1-ND; LCSC C28233 -> C136621; MPN (none) -> CL21B104KBFNNNE; Manufacturer (none) -> Samsung Electro-Mechanics
- C6: renamed from C5; Digi-Key_PN (none) -> 1276-1180-1-ND; LCSC C28233 -> C136621; MPN (none) -> CL21B104KBFNNNE; Manufacturer (none) -> Samsung Electro-Mechanics
- C7: renamed from C6; Digi-Key_PN (none) -> 1276-1180-1-ND; LCSC C28233 -> C136621; MPN (none) -> CL21B104KBFNNNE; Manufacturer (none) -> Samsung Electro-Mechanics
- C8: renamed from C7; Digi-Key_PN (none) -> 1276-1180-1-ND; LCSC C28233 -> C136621; MPN (none) -> CL21B104KBFNNNE; Manufacturer (none) -> Samsung Electro-Mechanics
- C9: renamed from C8; Digi-Key_PN (none) -> 1276-1180-1-ND; LCSC C28233 -> C136621; MPN (none) -> CL21B104KBFNNNE; Manufacturer (none) -> Samsung Electro-Mechanics
- D1: Digi-Key_PN (none) -> 3372-0805YGBD008S01TR-ND; MPN (none) -> 0805YGBD008S01; Manufacturer (none) -> CHANZON/BNDLIGHT/EKINGLUX
- EyeSPI1: Digi-Key_PN (none) -> 26-TF31-18S-0.5SH(800)CT-ND; MPN (none) -> TF31-18S-0.5SH(800); Manufacturer (none) -> Hirose Electric Co Ltd
- J1: Digi-Key_PN (none) -> SAM15543-ND; MPN (none) -> CES-113-02-T-D; Manufacturer (none) -> Samtec Inc.
- J10: Digi-Key_PN (none) -> SAM1035-04-ND; MPN (none) -> TSW-104-07-T-S; Manufacturer (none) -> Samtec Inc.
- J11: Digi-Key_PN (none) -> SAM1035-02-ND; MPN (none) -> TSW-102-07-T-S; Manufacturer (none) -> Samtec Inc.
- J2, J3, J4, J5: Digi-Key_PN (none) -> SAM15257-ND; MPN (none) -> SL-104-TT-19; Manufacturer (none) -> Samtec Inc.
- J6, J7, J8, J9: Digi-Key_PN (none) -> SL-106-TT-19-ND; MPN (none) -> SL-106-TT-19; Manufacturer (none) -> Samtec Inc.
- R1: renamed from R3; Digi-Key_PN (none) -> P680CCT-ND; LCSC C17798 -> C410034; MPN (none) -> ERJ-6ENF6800V; Manufacturer (none) -> Panasonic Electronic Components
- R10, R11, R4, R5, R6, R7, R8, R9: Digi-Key_PN (none) -> P330CCT-ND; LCSC C17630 -> C410007; MPN (none) -> ERJ-6ENF3300V; Manufacturer (none) -> Panasonic Electronic Components
- R2: renamed from R1; Digi-Key_PN (none) -> P330CCT-ND; LCSC C17630 -> C410007; MPN (none) -> ERJ-6ENF3300V; Manufacturer (none) -> Panasonic Electronic Components
- R3: renamed from R2; Digi-Key_PN (none) -> P330CCT-ND; LCSC C17630 -> C410007; MPN (none) -> ERJ-6ENF3300V; Manufacturer (none) -> Panasonic Electronic Components
- RN1: Digi-Key_PN (none) -> 118-4309R-101-100LF-ND; LCSC (none) -> C1360965; MPN (none) -> 4309R-101-100LF; Manufacturer (none) -> Bourns Inc.; Socket_Datasheet (none) -> https://app.adam-tech.com/products/download/data_sheet/2033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; Socket_PN (none) -> SMC-1-09-1-GT
- StemmaQT1: Digi-Key_PN (none) -> 455-1804-1-ND; LCSC C145956 -> C2764183; LCSC Part (none) -> C145956; MPN (none) -> SM04B-SRSS-TB(LF)(SN); Manufacturer (none) -> JST Sales America Inc.
- U1: Digi-Key_PN (none) -> 296-1568-5-ND; MPN (none) -> SN74HC05N; Manufacturer (none) -> Texas Instruments; Socket_Datasheet (none) -> http://www.on-shore.com/wp-content/uploads/2015/09/SAXXX0X0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; Socket_PN (none) -> SA143000
- U2: Digi-Key_PN (none) -> 296-1582-5-ND; MPN (none) -> SN74HC244N; Manufacturer (none) -> Texas Instruments; Socket_Datasheet (none) -> http://www.on-shore.com/wp-content/uploads/2015/09/SAXXX0X0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; Socket_PN (none) -> SA203000
Connections:
- net +3V3: now also Q1.1 (G), Q2.1 (G), Q3.1 (G), Q4.1 (G), Q5.1 (G), R13.1, R14.1, R16.1, R18.1, R20.1
- net +5V: now also C17.1, R15.1, R17.1, R19.1, U4.16 (VCC), U4.6 (G1)
- net CARDCS: now also EyeSPI1.10 (SD_CS), R24.2, R30.1
- net D4: now also U4.1 (A); no longer U2.6 (1A2)
- net D5: now also U4.2 (B); no longer U2.8 (1A3)
- net D6: now also U4.3 (C); no longer U2.17 (2A0)
- net GND: now also U2.17 (2A0), U2.6 (1A2), U2.8 (1A3), C17.2, R27.2, R28.2, R29.2, R30.2, R31.2, R32.2, U4.4 (G#2A), U4.5 (G#2B), U4.8 (GND)
- net MEM_CS: now also EyeSPI1.11 (MEM_CS), R25.2, R31.1
- net MISO: now also Q3.3 (D), R15.2; no longer EyeSPI1.6 (MISO), J8.3 (Pin_3), J9.3 (Pin_3)
- net MOSI: now also Q4.3 (D), R17.2; no longer EyeSPI1.5 (MOSI), J8.4 (Pin_4), J9.4 (Pin_4)
- net SCLK: now also Q5.3 (D), R19.2; no longer J8.5 (Pin_5), J9.5 (Pin_5)
- net TFTCS: now also EyeSPI1.9 (DISP_CS), R23.2, R29.1
- net TFTDC: now also EyeSPI1.7 (DC), R11.2
- net TSCS: now also EyeSPI1.12 (TS_CS), R26.2, R32.1
- net ~{CS3}: now also R21.1, U4.12 (Y3); no longer J8.6 (Pin_6), R11.2
- net ~{CS4}: now also R22.1, U4.15 (Y0); no longer J9.6 (Pin_6)
- net RNP2: now reaches J1.1 (Pin_1), U1.1, U1.3
- net RNP2: now also RN1.2 (R1); no longer RN1.4 (R3)
- net D1: now reaches J1.3 (Pin_3), RN1.6 (R5), U1.5
- net D0: now reaches J1.2 (Pin_2), U1.9
- net D0: now also RN1.7 (R6); no longer RN1.5 (R4)
- net STATUS: now reaches J1.13 (Pin_13), R2.1
- net ERROR: now reaches J1.15 (Pin_15), R3.1
- net RNP4: now reaches R2.2, U1.10
- net RNP4: now also RN1.4 (R3); no longer RN1.3 (R2)
- net RNP3: now reaches R3.2, U1.12
- net RNP3: now also RN1.3 (R2); no longer RN1.2 (R1)
- net RNP9: now reaches RN1.9 (R8)
- net RNP9: now also J2.4 (Pin_4), J3.4 (Pin_4), U1.11, U1.6, Q2.3 (D)
- net at U2.12 (1Y3): no longer R10.1
- net at U2.14 (1Y2): no longer R9.1
- net at U2.3 (2Y0): no longer R11.1
- net at U2.5 (2Y1): now also R11.1
- net SCK renamed SCLK3V
- net SCLK3V: now also J8.5 (Pin_5), J9.5 (Pin_5), Q5.2 (S), R20.2
- removed net SCL: EyeSPI1.13 (SCL), J2.4 (Pin_4), J3.4 (Pin_4), J4.4 (Pin_4), J5.4 (Pin_4), RN1.8 (R7), StemmaQT1.4 (SCL), U1.11, U1.6
- removed net SDA: EyeSPI1.14 (SDA), J2.3 (Pin_3), J3.3 (Pin_3), J4.3 (Pin_3), J5.3 (Pin_3), RN1.7 (R6), StemmaQT1.3 (SDA), U1.13, U1.8
- new net: R10.1, U4.10 (Y5)
- new net: R9.1, U4.9 (Y6)
- new net MISO3V: EyeSPI1.6 (MISO), J8.3 (Pin_3), J9.3 (Pin_3), Q3.2 (S), R16.2
- new net MOSI3V: EyeSPI1.5 (MOSI), J8.4 (Pin_4), J9.4 (Pin_4), Q4.2 (S), R18.2
- new net RNP5: RN1.5 (R4)
- new net RNP8: J2.3 (Pin_3), J3.3 (Pin_3), Q1.3 (D), RN1.8 (R7), U1.13, U1.8
- new net SCL3V: EyeSPI1.13 (SCL), J4.4 (Pin_4), J5.4 (Pin_4), Q2.2 (S), R14.2, StemmaQT1.4 (SCL)
- new net SDA3V: EyeSPI1.14 (SDA), J4.3 (Pin_3), J5.3 (Pin_3), Q1.2 (S), R13.2, StemmaQT1.3 (SDA)
- new net ~{CS3}-3V: J8.6 (Pin_6), R21.2, R27.1
- new net ~{CS4}-3V: J9.6 (Pin_6), R22.2, R28.1
- new net ~{CS5}: R23.1, U4.14 (Y1)
- new net ~{CS6}: R24.1, U4.13 (Y2)
- new net ~{CS7}: R25.1, U4.11 (Y4)
- new net ~{CS8}: R26.1, U4.7 (Y7)
- no-connect marks 27 -> 19
Other:
- note added: "Data Line Level Shifters"
- note removed: "D0"
- note removed: "D1"
- note removed: "ERROR"
- note removed: "STATUS"
- note removed: "STROBE"
- moved on the sheet: C1, C14, C15, C16, C2, C3, C4, C5, J10, J11, R10, R4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

Commit message: Enhanced 3D Models and render; Moved away from Tantalum footprint.
Parts:
- C1, C2, C3: footprint Capacitor_Tantalum_SMD:CP_EIA-3216-10_Kemet-I_Pad1.58x1.35mm_HandSolder -> Capacitor_SMD:C_0805_2012Metric_Pad1.18x1.45mm_HandSolder
Connections:
- net +5V: now also R15.2, R17.2; no longer R15.1, R17.1
- net CARDCS: now also R30.2; no longer R30.1
- net GND: now also R28.1, R29.1, R30.1, R32.1; no longer R28.2, R29.2, R30.2, R32.2
- net MISO: now also R15.1, R6.2; no longer R15.2, R6.1
- net MOSI: now also R17.1; no longer R17.2
- net RNP4: now also R2.1; no longer R2.2
- net STATUS: now also R2.2; no longer R2.1
- net TFTCS: now also R29.2; no longer R29.1
- net TFTDC: now also R11.1; no longer R11.2
- net TSCS: now also R32.2; no longer R32.1
- net ~{CS4}-3V: now also R28.2; no longer R28.1
- net at U2.13 (2A2): now also R6.1; no longer R6.2
- net at U2.5 (2Y1): now also R11.2; no longer R11.1
Other:
- moved on the sheet: R11, R15, R17, R2, R28, R29, R30, R32, R6
